Commit message: Rename flex_short->flex, fix assimp stl load bug
http://answers.ros.org/question/11569/planning_component_visualizer-bug/

File: urdf/fingers.urdf.xacro (robot description, xacro)
@@ -48,8 +48,8 @@
       <mimic joint="${mimic_source}" multiplier="${finger_flex_max}" offset="0.0" />
     </xacro:finger_flex_virtual>
-    <xacro:finger_flex_short parent="${name}_virtual_1_link" name="${name}_flex_1" reflect="${reflect}">
-      <origin xyz="${finger_d2} 0 0" rpy="0 0 0" />
-      <mimic joint="${mimic_source}" multiplier="${finger_flex_max}" offset="0.0" />
-    </xacro:finger_flex_short>
+    <xacro:finger_flex parent="${name}_virtual_1_link" name="${name}_flex_1" reflect="${reflect}">
+      <origin xyz="${finger_d2} 0 0" rpy="0 0 0" />
+      <mimic joint="${mimic_source}" multiplier="${finger_flex_max}" offset="0.0" />
+    </xacro:finger_flex>
     <!--Second flexor-->
     <xacro:finger_flex_virtual parent="${name}_flex_1_link" name="${name}_virtual_2" reflect="${reflect}">
@@ -57,8 +57,8 @@
       <mimic joint="${mimic_source}" multiplier="${finger_flex_max}" offset="0.0" />
     </xacro:finger_flex_virtual>
-    <xacro:finger_flex_short parent="${name}_virtual_2_link" name="${name}_flex_2" reflect="${reflect}">
-      <origin xyz="${finger_d2} 0 0" rpy="0 0 0" />
-      <mimic joint="${mimic_source}" multiplier="${finger_flex_max}" offset="0.0" />
-    </xacro:finger_flex_short>
+    <xacro:finger_flex parent="${name}_virtual_2_link" name="${name}_flex_2" reflect="${reflect}">
+      <origin xyz="${finger_d2} 0 0" rpy="0 0 0" />
+      <mimic joint="${mimic_source}" multiplier="${finger_flex_max}" offset="0.0" />
+    </xacro:finger_flex>
     <!--Third flexor-->
     <xacro:finger_flex_virtual parent="${name}_flex_2_link" name="${name}_virtual_3" reflect="${reflect}">
@@ -90,8 +90,8 @@
       <mimic joint="${mimic_source}" multiplier="${finger_flex_max}" offset="0.0" />
     </xacro:finger_flex_virtual>
-    <xacro:finger_flex_short parent="${name}_virtual_1_link" name="${name}_flex_1" reflect="${reflect}">
-      <origin xyz="${finger_d2} 0 0" rpy="0 0 0" />
-      <mimic joint="${mimic_source}" multiplier="${finger_flex_max}" offset="0.0" />
-    </xacro:finger_flex_short>
+    <xacro:finger_flex parent="${name}_virtual_1_link" name="${name}_flex_1" reflect="${reflect}">
+      <origin xyz="${finger_d2} 0 0" rpy="0 0 0" />
+      <mimic joint="${mimic_source}" multiplier="${finger_flex_max}" offset="0.0" />
+    </xacro:finger_flex>
     <!--Second flexor-->
     <xacro:finger_flex_virtual parent="${name}_flex_1_link" name="${name}_virtual_2" reflect="${reflect}">
@@ -232,5 +232,5 @@
     - origin: XML block containing the pose of the joint with respect to its parent
   -->
-  <xacro:macro name="finger_flex_short" params="name parent reflect *origin *mimic">
+  <xacro:macro name="finger_flex" params="name parent reflect *origin *mimic">
     <joint name="${name}_joint" type="revolute">
       <parent link="${parent}" />
@@ -252,12 +252,12 @@
         <origin xyz="0 0 0" rpy="0 0 0" />
         <geometry>
-          <mesh filename="package://hey5_description/meshes/finger_flex_short${vis_suffix}.stl" />
-        </geometry>
-        <material name="Hey5DarkGrey" />
-      </visual>
-      <collision>
-        <origin xyz="0 0 0" rpy="0 0 0" />
-        <geometry>
-          <mesh filename="package://hey5_description/meshes/finger_flex_short_collision.stl" />
+          <mesh filename="package://hey5_description/meshes/finger_flex${vis_suffix}.stl" />
+        </geometry>
+        <material name="Hey5DarkGrey" />
+      </visual>
+      <collision>
+        <origin xyz="0 0 0" rpy="0 0 0" />
+        <geometry>
+          <mesh filename="package://hey5_description/meshes/finger_flex_collision.stl" />
         </geometry>
       </collision>

Commit message: Default to use collision meshes

File: urdf/fingers.urdf.xacro (robot description, xacro)
@@ -28,5 +28,5 @@
     collision meshes for visualization as well
   -->
-  <xacro:property name="vis_suffix"  value="" />
+  <xacro:property name="vis_suffix"  value="_collision" />
   <!--
     Create one non-thumb finger with one abduction/adduction joint and three

Commit message: Remove usage of mimic joints

File: urdf/fingers.urdf.xacro (robot description, xacro)
@@ -38,5 +38,5 @@
     - origin: XML block containing the pose of the first finger joint with respect to its parent
   -->
-  <xacro:macro name="finger" params="name parent reflect *origin mimic_source">
+  <xacro:macro name="finger" params="name parent reflect *origin">
     <!--Abductor-->
     <xacro:finger_abd parent="${parent}" name="${name}_abd" reflect="${reflect}">
@@ -46,27 +46,21 @@
     <xacro:finger_flex_virtual parent="${name}_abd_link" name="${name}_virtual_1" reflect="${reflect}">
       <origin xyz="${finger_d1} 0 0" rpy="${reflect * 90 * deg_to_rad} 0 0" />
-      <mimic joint="${mimic_source}" multiplier="${finger_flex_max}" offset="0.0" />
     </xacro:finger_flex_virtual>
     <xacro:finger_flex parent="${name}_virtual_1_link" name="${name}_flex_1" reflect="${reflect}">
       <origin xyz="${finger_d2} 0 0" rpy="0 0 0" />
-      <mimic joint="${mimic_source}" multiplier="${finger_flex_max}" offset="0.0" />
     </xacro:finger_flex>
     <!--Second flexor-->
     <xacro:finger_flex_virtual parent="${name}_flex_1_link" name="${name}_virtual_2" reflect="${reflect}">
       <origin xyz="${finger_d1} 0 0" rpy="0 0 0" />
-      <mimic joint="${mimic_source}" multiplier="${finger_flex_max}" offset="0.0" />
     </xacro:finger_flex_virtual>
     <xacro:finger_flex parent="${name}_virtual_2_link" name="${name}_flex_2" reflect="${reflect}">
       <origin xyz="${finger_d2} 0 0" rpy="0 0 0" />
-      <mimic joint="${mimic_source}" multiplier="${finger_flex_max}" offset="0.0" />
     </xacro:finger_flex>
     <!--Third flexor-->
     <xacro:finger_flex_virtual parent="${name}_flex_2_link" name="${name}_virtual_3" reflect="${reflect}">
       <origin xyz="${finger_d1} 0 0" rpy="0 0 0" />
-      <mimic joint="${mimic_source}" multiplier="${finger_flex_max}" offset="0.0" />
     </xacro:finger_flex_virtual>
     <xacro:finger_flex_tip parent="${name}_virtual_3_link" name="${name}_flex_3" reflect="${reflect}">
       <origin xyz="${finger_d2} 0 0" rpy="0 0 0" />
-      <mimic joint="${mimic_source}" multiplier="${finger_flex_max}" offset="0.0" />
     </xacro:finger_flex_tip>
   </xacro:macro>
@@ -80,5 +74,5 @@
     - origin: XML block containing the pose of the first finger joint with respect to its parent
   -->
-  <xacro:macro name="thumb" params="name parent reflect *origin mimic_source">
+  <xacro:macro name="thumb" params="name parent reflect *origin">
     <!--Abductor-->
     <xacro:thumb_abd parent="${parent}" name="${name}_abd" reflect="${reflect}">
@@ -88,18 +82,14 @@
     <xacro:finger_flex_virtual parent="${name}_abd_link" name="${name}_virtual_1" reflect="${reflect}">
       <origin xyz="${0.0355 - finger_d2} 0.0033 0" rpy="${-reflect * 65.56 * deg_to_rad} 0 0" />
-      <mimic joint="${mimic_source}" multiplier="${finger_flex_max}" offset="0.0" />
     </xacro:finger_flex_virtual>
     <xacro:finger_flex parent="${name}_virtual_1_link" name="${name}_flex_1" reflect="${reflect}">
       <origin xyz="${finger_d2} 0 0" rpy="0 0 0" />
-      <mimic joint="${mimic_source}" multiplier="${finger_flex_max}" offset="0.0" />
     </xacro:finger_flex>
     <!--Second flexor-->
     <xacro:finger_flex_virtual parent="${name}_flex_1_link" name="${name}_virtual_2" reflect="${reflect}">
       <origin xyz="${finger_d1} 0 0" rpy="0 0 0" />
-      <mimic joint="${mimic_source}" multiplier="${finger_flex_max}" offset="0.0" />
     </xacro:finger_flex_virtual>
     <xacro:finger_flex_tip parent="${name}_virtual_2_link" name="${name}_flex_2" reflect="${reflect}">
       <origin xyz="${finger_d2} 0 0" rpy="0 0 0" />
-      <mimic joint="${mimic_source}" multiplier="${finger_flex_max}" offset="0.0" />
     </xacro:finger_flex_tip>
   </xacro:macro>
@@ -191,5 +181,5 @@
     - origin: XML block containing the pose of the joint with respect to its parent
   -->
-  <xacro:macro name="finger_flex_virtual" params="name parent reflect *origin *mimic" >
+  <xacro:macro name="finger_flex_virtual" params="name parent reflect *origin" >
     <joint name="${name}_joint" type="revolute">
       <parent link="${parent}" />
@@ -199,5 +189,4 @@
       <limit lower="${finger_flex_min}" upper="${finger_flex_max}" effort="${finger_max_eff}" velocity="${finger_max_vel}" />
       <dynamics friction="${finger_friction}" damping="${finger_damping}"/>
-      <insert_block name="mimic" />
     </joint>
     <link name="${name}_link">
@@ -232,5 +221,5 @@
     - origin: XML block containing the pose of the joint with respect to its parent
   -->
-  <xacro:macro name="finger_flex" params="name parent reflect *origin *mimic">
+  <xacro:macro name="finger_flex" params="name parent reflect *origin">
     <joint name="${name}_joint" type="revolute">
       <parent link="${parent}" />
@@ -240,5 +229,4 @@
       <limit lower="${finger_flex_min}" upper="${finger_flex_max}" effort="${finger_max_eff}" velocity="${finger_max_vel}" />
       <dynamics friction="${finger_friction}" damping="${finger_damping}"/>
-      <insert_block name="mimic" />
     </joint>
     <link name="${name}_link">
@@ -274,5 +262,5 @@
     - origin: XML block containing the pose of the joint with respect to its parent
   -->
-  <xacro:macro name="finger_flex_tip" params="name parent reflect *origin *mimic">
+  <xacro:macro name="finger_flex_tip" params="name parent reflect *origin">
     <joint name="${name}_joint" type="revolute">
       <parent link="${parent}" />
@@ -282,5 +270,4 @@
       <limit lower="${finger_flex_min}" upper="${finger_flex_max}" effort="${finger_max_eff}" velocity="${finger_max_vel}" />
       <dynamics friction="${finger_friction}" damping="${finger_damping}"/>
-      <insert_block name="mimic" />
     </joint>
     <link name="${name}_link">

File: urdf/hey5_hand.urdf.xacro (robot description, xacro)
@@ -13,21 +13,10 @@
   <xacro:include filename="$(find hey5_description)/urdf/fingers.urdf.xacro" />
   <xacro:include filename="$(find hey5_description)/urdf/palm.urdf.xacro" />
-  <!--Command source. TODO: Remove!-->
-  <xacro:macro name="cmd_source" params="name parent *origin">
-    <joint name="${name}_joint" type="revolute">
-      <parent link="${parent}" />
-      <child link="${name}_link" />
-      <insert_block name="origin" />
-      <axis xyz="0 0 1" />
-      <limit lower="0.0" upper="1.0" effort="10.0" velocity="20.0" /> <!--TODO: Check-->
-      <!--TODO: Add joint dynamics?-->
-    </joint>
-    <link name="${name}_link">
-      <inertial>
-        <mass value="0.01" /> <!--TODO: can we make it zero and still have a stable dynamic simulation?-->
-        <inertia ixx="0" ixy="0" ixz="0" iyy="0" iyz="0" izz="0" />
-      </inertial>
-    </link>
-  </xacro:macro>
+  <!--Constants-->
+  <xacro:property name="thumb_act_flex_start"  value="2.0" />
+  <xacro:property name="index_act_flex_start"  value="0.7" />
+  <xacro:property name="middle_act_flex_start" value="0.0" />
+  <xacro:property name="ring_act_flex_start"   value="0.75" />
+  <xacro:property name="little_act_flex_start" value="0.75" />
   <!--
     Create a complete hey5 hand (right or left).
@@ -43,15 +32,5 @@
       <insert_block name="origin" />
     </xacro:palm>
-    <!--Command sources-->
-<!--    <xacro:cmd_source parent="${name}_palm_link" name="${name}_thumb" >
-      <origin xyz="0.05 0 0" rpy="0 0 0" />
-    </xacro:cmd_source>
-    <xacro:cmd_source parent="${name}_palm_link" name="${name}_index" >
-      <origin xyz="0.05 0 0" rpy="0 0 0" />
-    </xacro:cmd_source>
-    <xacro:cmd_source parent="${name}_palm_link" name="${name}_mrl" >
-      <origin xyz="0.05 0 0" rpy="0 0 0" />
-    </xacro:cmd_source>-->
-    <!-- Actuators -->
+    <!--Actuators-->
     <xacro:thumb_actuator parent="${name}_palm_link" name="${name}_thumb">
       <origin xyz="0 0 0" rpy="0 0 0" /> <!-- TODO: Change! -->
@@ -65,17 +44,17 @@
     <!--Fingers-->
     <!-- TODO: Add grasp hack? -->
-    <xacro:thumb parent="${name}_palm_link" name="${name}_thumb" reflect="${reflect}" mimic_source="${name}_thumb_joint">
+    <xacro:thumb parent="${name}_palm_link" name="${name}_thumb" reflect="${reflect}">
       <origin xyz="0.0911 0.0132 ${reflect * 0.038}" rpy="0 ${-reflect * 65 * deg_to_rad} 0" />
     </xacro:thumb>
-    <xacro:finger parent="${name}_palm_link" name="${name}_index" reflect="${reflect}" mimic_source="${name}_index_joint">
+    <xacro:finger parent="${name}_palm_link" name="${name}_index" reflect="${reflect}">
       <origin xyz="0.1265 0.00399 ${reflect * 0.0265}" rpy="${-reflect * 90 * deg_to_rad} ${-reflect * 15 * deg_to_rad} 0" />
     </xacro:finger>
-    <xacro:finger parent="${name}_palm_link" name="${name}_middle" reflect="${reflect}" mimic_source="${name}_mrl_joint">
+    <xacro:finger parent="${name}_palm_link" name="${name}_middle" reflect="${reflect}">
       <origin xyz="0.1335 0.00399 ${reflect * 0.007}" rpy="${-reflect * 90 * deg_to_rad} 0 0" />
     </xacro:finger>
-    <xacro:finger parent="${name}_palm_link" name="${name}_ring" reflect="${reflect}" mimic_source="${name}_mrl_joint">
+    <xacro:finger parent="${name}_palm_link" name="${name}_ring" reflect="${reflect}">
       <origin xyz="0.1265 0.00399 ${reflect * -0.0125}" rpy="${-reflect * 90 * deg_to_rad} ${reflect * 5 * deg_to_rad} 0" />
     </xacro:finger>
-    <xacro:finger parent="${name}_palm_link" name="${name}_little" reflect="${reflect}" mimic_source="${name}_mrl_joint">
+    <xacro:finger parent="${name}_palm_link" name="${name}_little" reflect="${reflect}">
       <origin xyz="0.1165 0.00399 ${reflect * -0.032}" rpy="${-reflect * 90 * deg_to_rad} ${reflect * 15 * deg_to_rad} 0" />
     </xacro:finger>

Commit message: Minor dimension tweaks to harmonize with docs, CAD

File: urdf/fingers.urdf.xacro (robot description, xacro)
@@ -81,5 +81,5 @@
     <!--First flexor-->
     <xacro:finger_flex_virtual parent="${name}_abd_link" name="${name}_virtual_1" reflect="${reflect}">
-      <origin xyz="${0.0355 - finger_d2} 0.0033 0" rpy="${-reflect * 65.56 * deg_to_rad} 0 0" />
+      <origin xyz="${0.0355 - finger_d2} 0.003 0" rpy="${-reflect * 65.56 * deg_to_rad} 0 0" />
     </xacro:finger_flex_virtual>
     <xacro:finger_flex parent="${name}_virtual_1_link" name="${name}_flex_1" reflect="${reflect}">

File: urdf/hey5_hand.urdf.xacro (robot description, xacro)
@@ -46,17 +46,17 @@
     <!-- TODO: Add grasp hack? -->
     <xacro:thumb parent="${name}_palm_link" name="${name}_thumb" reflect="${reflect}">
-      <origin xyz="0.0911 0.0132 ${reflect * 0.038}" rpy="0 ${-reflect * 65 * deg_to_rad} 0" />
+      <origin xyz="0.0901 0.0134 ${reflect * 0.038}" rpy="0 ${-reflect * 65 * deg_to_rad} 0" />
     </xacro:thumb>
     <xacro:finger parent="${name}_palm_link" name="${name}_index" reflect="${reflect}">
-      <origin xyz="0.1265 0.00399 ${reflect * 0.0265}" rpy="${-reflect * 90 * deg_to_rad} ${-reflect * 30 * deg_to_rad} 0" />
+      <origin xyz="0.1265 0.0042 ${reflect * 0.0265}" rpy="${-reflect * 90 * deg_to_rad} ${-reflect * 30 * deg_to_rad} 0" />
     </xacro:finger>
     <xacro:finger parent="${name}_palm_link" name="${name}_middle" reflect="${reflect}">
-      <origin xyz="0.1335 0.00399 ${reflect * 0.007}" rpy="${-reflect * 90 * deg_to_rad} 0 0" />
+      <origin xyz="0.1335 0.0042 ${reflect * 0.007}" rpy="${-reflect * 90 * deg_to_rad} 0 0" />
     </xacro:finger>
     <xacro:finger parent="${name}_palm_link" name="${name}_ring" reflect="${reflect}">
-      <origin xyz="0.1265 0.00399 ${reflect * -0.0125}" rpy="${-reflect * 90 * deg_to_rad} ${reflect * 15 * deg_to_rad} 0" />
+      <origin xyz="0.1265 0.0042 ${reflect * -0.0125}" rpy="${-reflect * 90 * deg_to_rad} ${reflect * 15 * deg_to_rad} 0" />
     </xacro:finger>
     <xacro:finger parent="${name}_palm_link" name="${name}_little" reflect="${reflect}">
-      <origin xyz="0.1165 0.00399 ${reflect * -0.032}" rpy="${-reflect * 90 * deg_to_rad} ${reflect * 30 * deg_to_rad} 0" />
+      <origin xyz="0.1165 0.0042 ${reflect * -0.032}" rpy="${-reflect * 90 * deg_to_rad} ${reflect * 30 * deg_to_rad} 0" />
     </xacro:finger>
     <!--Transmissions-->

Commit message: Add gazebo references with black material

File: urdf/fingers.urdf.xacro (robot description, xacro)
@@ -131,4 +131,7 @@
       </collision>
     </link>
+    <gazebo reference="${name}_link">
+      <material>Gazebo/Black</material>
+    </gazebo>
   </xacro:macro>
   <!--
@@ -169,4 +172,7 @@
       </collision>
     </link>
+    <gazebo reference="${name}_link">
+      <material>Gazebo/Black</material>
+    </gazebo>
   </xacro:macro>
   <!--
@@ -208,4 +214,7 @@
       </collision>
     </link>
+    <gazebo reference="${name}_link">
+      <material>Gazebo/Black</material>
+    </gazebo>
   </xacro:macro>
   <!--
@@ -248,4 +257,7 @@
       </collision>
     </link>
+    <gazebo reference="${name}_link">
+      <material>Gazebo/Black</material>
+    </gazebo>
   </xacro:macro>
   <!--
@@ -288,4 +300,7 @@
       </collision>
     </link>
+    <gazebo reference="${name}_link">
+      <material>Gazebo/Black</material>
+    </gazebo>
   </xacro:macro>
 </robot>

File: urdf/palm.urdf.xacro (robot description, xacro)
@@ -44,4 +44,7 @@
       </collision>
     </link>
+    <gazebo reference="${name}_link">
+      <material>Gazebo/Black</material>
+    </gazebo>
   </xacro:macro>
 </robot>
