Commit message: Add hand_grasping_frame

File: urdf/hey5_hand.urdf.xacro (robot description, xacro)
@@ -106,4 +106,11 @@
       flex_reduction="${36 * deg_to_rad / (530 * deg_to_rad - little_act_flex_start)}"
     />
+    <link name="${name}_grasping_frame"/>
+    <joint name="${name}_grasping_fixed_joint" type="fixed">
+      <parent link="${name}_palm_link"/>
+      <child link="${name}_grasping_frame"/>
+      <axis xyz="0 0 1" />
+      <origin xyz="0.13 0.02 0" rpy="0 0 0"/>
+    </joint>
   </xacro:macro>
 </robot>

Commit message: Update hand transmissions, fully open config
- Add some overlap between abduction and flexion to more closely mimic
  hardware

- Spread fingers more on fully open configuration

File: urdf/hey5_hand.urdf.xacro (robot description, xacro)
@@ -49,5 +49,5 @@
     </xacro:thumb>
     <xacro:finger parent="${name}_palm_link" name="${name}_index" reflect="${reflect}">
-      <origin xyz="0.1265 0.00399 ${reflect * 0.0265}" rpy="${-reflect * 90 * deg_to_rad} ${-reflect * 15 * deg_to_rad} 0" />
+      <origin xyz="0.1265 0.00399 ${reflect * 0.0265}" rpy="${-reflect * 90 * deg_to_rad} ${-reflect * 30 * deg_to_rad} 0" />
     </xacro:finger>
     <xacro:finger parent="${name}_palm_link" name="${name}_middle" reflect="${reflect}">
@@ -55,8 +55,8 @@
     </xacro:finger>
     <xacro:finger parent="${name}_palm_link" name="${name}_ring" reflect="${reflect}">
-      <origin xyz="0.1265 0.00399 ${reflect * -0.0125}" rpy="${-reflect * 90 * deg_to_rad} ${reflect * 5 * deg_to_rad} 0" />
+      <origin xyz="0.1265 0.00399 ${reflect * -0.0125}" rpy="${-reflect * 90 * deg_to_rad} ${reflect * 15 * deg_to_rad} 0" />
     </xacro:finger>
     <xacro:finger parent="${name}_palm_link" name="${name}_little" reflect="${reflect}">
-      <origin xyz="0.1165 0.00399 ${reflect * -0.032}" rpy="${-reflect * 90 * deg_to_rad} ${reflect * 15 * deg_to_rad} 0" />
+      <origin xyz="0.1165 0.00399 ${reflect * -0.032}" rpy="${-reflect * 90 * deg_to_rad} ${reflect * 30 * deg_to_rad} 0" />
     </xacro:finger>
     <!--Transmissions-->
@@ -67,5 +67,5 @@
       jnt_abd_start="${0.0 * deg_to_rad}"
       jnt_abd_stop="${90 * deg_to_rad}"
-      abd_reduction="${90 * deg_to_rad / thumb_act_flex_start}"
+      abd_reduction="${75 * deg_to_rad / thumb_act_flex_start}"
       flex_reduction="${40 * deg_to_rad / (360 * deg_to_rad - thumb_act_flex_start)}"
     />
@@ -75,6 +75,6 @@
       act_flex_start="${index_act_flex_start}"
       jnt_abd_start="${0.0 * deg_to_rad}"
-      jnt_abd_stop="${15.0 * deg_to_rad}"
-      abd_reduction="${15.0 * deg_to_rad / index_act_flex_start}"
+      jnt_abd_stop="${30.0 * deg_to_rad}"
+      abd_reduction="${20.0 * deg_to_rad / index_act_flex_start}"
       flex_reduction="${36 * deg_to_rad / (390 * deg_to_rad - index_act_flex_start)}"
     />
@@ -92,7 +92,7 @@
       act_name="${name}_mrl_motor"
       act_flex_start="${ring_act_flex_start}"
-      jnt_abd_start="${-2.5 * deg_to_rad}"
+      jnt_abd_start="${-15.0 * deg_to_rad}"
       jnt_abd_stop="${0.0 * deg_to_rad}"
-      abd_reduction="${-2.5 * deg_to_rad / ring_act_flex_start}"
+      abd_reduction="${-10.0 * deg_to_rad / ring_act_flex_start}"
       flex_reduction="${36 * deg_to_rad / (530 * deg_to_rad - ring_act_flex_start)}"
     />
@@ -101,7 +101,7 @@
       act_name="${name}_mrl_motor"
       act_flex_start="${little_act_flex_start}"
-      jnt_abd_start="${-5.0 * deg_to_rad}"
+      jnt_abd_start="${-30.0 * deg_to_rad}"
       jnt_abd_stop="${0.0 * deg_to_rad}"
-      abd_reduction="${-5.0 * deg_to_rad / little_act_flex_start}"
+      abd_reduction="${-20.0 * deg_to_rad / little_act_flex_start}"
       flex_reduction="${36 * deg_to_rad / (530 * deg_to_rad - little_act_flex_start)}"
     />

Commit message: Add hand_tool_link

File: urdf/hey5_hand.urdf.xacro (robot description, xacro)
@@ -30,4 +30,20 @@
   -->
   <xacro:macro name="hey5_hand" params="name parent reflect *origin">
+  <!-- Tool Link -->
+    <link name="${name}_tool_link">
+      <inertial>
+        <origin xyz="0 0 0" rpy="0 0 0" />
+        <mass value="0.0001" />
+        <inertia ixx="0.00001" ixy="0.0" ixz="0.0"
+                 iyy="0.00001" iyz="0.0"
+                 izz="0.00001" />
+      </inertial>
+    </link>
+    <joint name="${name}_tool_joint" type="fixed">
+      <insert_block name="origin"/>
+      <parent link="${parent}" />
+      <child link="${name}_tool_link" />
+       <axis xyz="0 0 0" />
+    </joint>
     <!--Palm-->
     <xacro:palm parent="${parent}" name="${name}_palm" reflect="${reflect}" >
