Commit message: Update material specification
- Make whole hand dark grey
- Use unique material names to prevent clashes when composing models

File: urdf/actuators.urdf.xacro (robot description, xacro)
@@ -35,5 +35,5 @@
           <sphere radius="0.001"/>
         </geometry>
-        <material name="LightGrey" />
+        <material name="Hey5DarkGrey" />
       </visual>
       <collision>
@@ -73,5 +73,5 @@
           <sphere radius="0.001"/>
         </geometry>
-        <material name="LightGrey" />
+        <material name="Hey5DarkGrey" />
       </visual>
       <collision>
@@ -111,5 +111,5 @@
           <sphere radius="0.001"/>
         </geometry>
-        <material name="LightGrey" />
+        <material name="Hey5DarkGrey" />
       </visual>
       <collision>
@@ -145,5 +145,5 @@
           <sphere radius="0.001"/>
         </geometry>
-        <material name="LightGrey" />
+        <material name="Hey5DarkGrey" />
       </visual>
       <collision>

File: urdf/fingers.urdf.xacro (robot description, xacro)
@@ -133,5 +133,5 @@
           <mesh filename="package://hey5_description/meshes/finger_abd${vis_suffix}.stl" scale="1 1 ${reflect}" />
         </geometry>
-        <material name="DarkGrey" />
+        <material name="Hey5DarkGrey" />
       </visual>
       <collision>
@@ -172,5 +172,5 @@
           <mesh filename="package://hey5_description/meshes/thumb_abd${vis_suffix}.stl" scale="1 1 ${reflect}" />
         </geometry>
-        <material name="DarkGrey" />
+        <material name="Hey5DarkGrey" />
       </visual>
       <collision>
@@ -212,5 +212,5 @@
           <box size="${finger_d2} 0.002 0.012" />
         </geometry>
-        <material name="DarkGrey" />
+        <material name="Hey5DarkGrey" />
       </visual>
       <collision>
@@ -254,5 +254,5 @@
           <mesh filename="package://hey5_description/meshes/finger_flex_short${vis_suffix}.stl" />
         </geometry>
-        <material name="DarkGrey" />
+        <material name="Hey5DarkGrey" />
       </visual>
       <collision>
@@ -296,5 +296,5 @@
           <mesh filename="package://hey5_description/meshes/finger_flex_tip${vis_suffix}.stl" />
         </geometry>
-        <material name="DarkGrey" />
+        <material name="Hey5DarkGrey" />
       </visual>
       <collision>

File: urdf/materials.urdf.xacro (robot description, xacro)
@@ -8,11 +8,5 @@
 -->
 <robot>
-  <material name="Grey">
-    <color rgba="0.7 0.7 0.7 1.0"/>
-  </material>
-  <material name="LightGrey">
-    <color rgba="0.9 0.9 0.9 1.0"/>
-  </material>
- <material name="DarkGrey">
+ <material name="Hey5DarkGrey">
    <color rgba="0.2 0.2 0.2 1.0"/>
  </material>

File: urdf/palm.urdf.xacro (robot description, xacro)
@@ -34,5 +34,5 @@
           <mesh filename="package://hey5_description/meshes/palm.stl" scale="1 1 ${reflect}" />
         </geometry>
-        <material name="LightGrey" />
+        <material name="Hey5DarkGrey" />
       </visual>
       <collision>

Commit message: Leverage macro for common actuator implementation

File: urdf/actuators.urdf.xacro (robot description, xacro)
@@ -9,119 +9,38 @@
 <robot xmlns:xacro="http://ros.org/wiki/xacro">
 <!-- TODO: Doc macros. Also doc created values. Applies also to finger macros. -->
-  <!-- Thumb -->
+  <!-- Thumb actuator -->
   <xacro:macro name="thumb_actuator" params="name parent *origin">
-    <joint name="${name}_joint" type="revolute">
-      <parent link="${parent}" />
-      <child link="${name}_link" />
+    <xacro:actuator_impl parent="${parent}" name="${name}">
       <insert_block name="origin" />
-      <axis xyz="0 0 1" />
       <limit lower="${-150 * deg_to_rad}" upper="${360 * deg_to_rad}" effort="2.0" velocity="3.35" /> <!-- TODO: Tune effort -->
-      <dynamics friction="0.0" damping="0.5"/> <!-- TODO: Tune -->
-      <!-- TODO: Tune -->
       <safety_controller k_position="20"
                          k_velocity="20"
                          soft_lower_limit="${-150.0 * deg_to_rad}"
                          soft_upper_limit="${ 360.0 * deg_to_rad}" />
-    </joint>
-    <link name="${name}_link">
-      <inertial>
-        <origin xyz="0 0 0" rpy="0 0 0" />
-        <mass value="0.05" /> <!--TODO: can we make it zero and still have a stable dynamic simulation?-->
-        <inertia ixx="0" ixy="0" ixz="0" iyy="0" iyz="0" izz="0" />
-      </inertial>
-      <visual>
-        <origin xyz="0 0 0" rpy="0 0 0" />
-        <geometry>
-          <sphere radius="0.001"/>
-        </geometry>
-        <material name="Hey5DarkGrey" />
-      </visual>
-      <collision>
-        <origin xyz="0 0 0" rpy="0 0 0" />
-        <geometry>
-          <sphere radius="0.001"/>
-        </geometry>
-      </collision>
-    </link>
-    <!-- TODO: Add grasp hack -->
-    <xacro:position_reducer name="${name}" reduction="1.0"/>
+    </xacro:actuator_impl>
   </xacro:macro>
-  <!-- Index -->
+  <!-- Index actuator -->
   <xacro:macro name="index_actuator" params="name parent *origin">
-    <joint name="${name}_joint" type="revolute">
-      <parent link="${parent}" />
-      <child link="${name}_link" />
+    <xacro:actuator_impl parent="${parent}" name="${name}">
       <insert_block name="origin" />
-      <axis xyz="0 0 1" />
       <limit lower="${-175 * deg_to_rad}" upper="${390 * deg_to_rad}" effort="2.0" velocity="3.35" /> <!-- TODO: Tune effort -->
-      <dynamics friction="0.0" damping="0.5"/> <!-- TODO: Tune -->
-      <!-- TODO: Tune -->
       <safety_controller k_position="20"
                          k_velocity="20"
                          soft_lower_limit="${-175.0 * deg_to_rad}"
                          soft_upper_limit="${ 390.0 * deg_to_rad}" />
-    </joint>
-    <link name="${name}_link">
-      <inertial>
-        <origin xyz="0 0 0" rpy="0 0 0" />
-        <mass value="0.05" /> <!--TODO: can we make it zero and still have a stable dynamic simulation?-->
-        <inertia ixx="0" ixy="0" ixz="0" iyy="0" iyz="0" izz="0" />
-      </inertial>
-      <visual>
-        <origin xyz="0 0 0" rpy="0 0 0" />
-        <geometry>
-          <sphere radius="0.001"/>
-        </geometry>
-        <material name="Hey5DarkGrey" />
-      </visual>
-      <collision>
-        <origin xyz="0 0 0" rpy="0 0 0" />
-        <geometry>
-          <sphere radius="0.001"/>
-        </geometry>
-      </collision>
-    </link>
-    <!-- TODO: Add grasp hack -->
-    <xacro:position_reducer name="${name}" reduction="1.0"/>
+    </xacro:actuator_impl>
   </xacro:macro>
-    <!-- Middle, ring, little (mrl) -->
+  <!-- Middle, ring, little (mrl) actuator -->
   <xacro:macro name="mrl_actuator" params="name parent *origin">
-    <joint name="${name}_joint" type="revolute">
-      <parent link="${parent}" />
-      <child link="${name}_link" />
+    <xacro:actuator_impl parent="${parent}" name="${name}">
       <insert_block name="origin" />
-      <axis xyz="0 0 1" />
       <limit lower="${-145 * deg_to_rad}" upper="${530 * deg_to_rad}" effort="2.0" velocity="3.56" /> <!-- TODO: Tune effort -->
-      <dynamics friction="0.0" damping="0.5"/> <!-- TODO: Tune -->
-      <!-- TODO: Tune -->
       <safety_controller k_position="20"
                          k_velocity="20"
                          soft_lower_limit="${-145 * deg_to_rad}"
                          soft_upper_limit="${ 530 * deg_to_rad}" />
-    </joint>
-    <link name="${name}_link">
-      <inertial>
-        <origin xyz="0 0 0" rpy="0 0 0" />
-        <mass value="0.05" /> <!--TODO: can we make it zero and still have a stable dynamic simulation?-->
-        <inertia ixx="0" ixy="0" ixz="0" iyy="0" iyz="0" izz="0" />
-      </inertial>
-      <visual>
-        <origin xyz="0 0 0" rpy="0 0 0" />
-        <geometry>
-          <sphere radius="0.001"/>
-        </geometry>
-        <material name="Hey5DarkGrey" />
-      </visual>
-      <collision>
-        <origin xyz="0 0 0" rpy="0 0 0" />
-        <geometry>
-          <sphere radius="0.001"/>
-        </geometry>
-      </collision>
-    </link>
-    <!-- TODO: Add grasp hack -->
-    <xacro:position_reducer name="${name}" reduction="1.0"/>
+    </xacro:actuator_impl>
   </xacro:macro>
-  <!-- Common actuator implementation. TODO: Can we double-forward the origin block? -->
+  <!-- Common actuator implementation -->
   <xacro:macro name="actuator_impl" params="name parent *origin *limit *safety_controller">
     <joint name="${name}_joint" type="revolute">
@@ -155,5 +74,4 @@
     </link>
     <xacro:position_reducer name="${name}" reduction="1.0"/>
-    <!-- TODO: Add grasp hack -->
   </xacro:macro>
  <!-- Position joint reducer -->

Commit message: Update hand inertial properties
- Inertia tensors for all links except palm are approximately four
  orders of magnitude larger to prevent the Gazebo simulation from
  becoming unstable.

- Palm mass is lower to take into account that actuator mass is
  specified separately.

File: urdf/actuators.urdf.xacro (robot description, xacro)
@@ -63,6 +63,6 @@
       <inertial>
         <origin xyz="0 0 0" rpy="0 0 0" />
-        <mass value="0.05" /> <!--TODO: can we make it zero and still have a stable dynamic simulation?-->
-        <inertia ixx="0" ixy="0" ixz="0" iyy="0" iyz="0" izz="0" />
+        <mass value="0.05" />
+        <inertia ixx="0.001" ixy="0" ixz="0" iyy="0.001" iyz="0" izz="0.001" /> <!--To stabilize simulation-->
       </inertial>
       <visual>

File: urdf/fingers.urdf.xacro (robot description, xacro)
@@ -115,6 +115,5 @@
         <origin xyz="-0.0018 0.0 0.0028" rpy="0 0 0" />
         <mass value="0.018" />
-        <inertia ixx="0.000000360" ixy="0.000000000" ixz="-0.000000059"
-                 iyy="0.000000808" iyz="0.000000000" izz="0.000000640" />
+        <inertia ixx="0.001" ixy="0" ixz="0" iyy="0.001" iyz="0" izz="0.001" /> <!-- To stabilize simulation -->
       </inertial>
       <visual>
@@ -154,6 +153,5 @@
         <origin xyz="-0.0132 0.0037 -0.0017" rpy="0 0 0" />
         <mass value="0.014" />
-        <inertia ixx="0.000000290" ixy="0.000000078" ixz="-0.000000035"
-                 iyy="0.000000995" iyz="-0.000000020" izz="0.000000955" />
+        <inertia ixx="0.001" ixy="0" ixz="0" iyy="0.001" iyz="0" izz="0.001" /> <!-- To stabilize simulation -->
       </inertial>
       <visual>
@@ -194,5 +192,5 @@
         <origin xyz="${finger_d2 / 2.0} 0 0" rpy="0 0 0" />
         <mass value="0.01" /> <!--TODO: can we make it zero and still have a stable dynamic simulation?-->
-        <inertia ixx="0" ixy="0" ixz="0" iyy="0" iyz="0" izz="0" />
+        <inertia ixx="0.001" ixy="0" ixz="0" iyy="0.001" iyz="0" izz="0.001" /> <!-- To stabilize simulation -->
       </inertial>
       <visual>
@@ -234,6 +232,5 @@
         <origin xyz="0.0047 0.0031 0.0" rpy="0 0 0" />
         <mass value="0.009" />
-        <inertia ixx="0.000000143" ixy="0.000000007" ixz="0.000000000"
-                 iyy="0.000000228" iyz="0.000000000" izz="0.000000232" />
+        <inertia ixx="0.001" ixy="0" ixz="0" iyy="0.001" iyz="0" izz="0.001" /> <!-- To stabilize simulation -->
       </inertial>
       <visual>
@@ -275,6 +272,5 @@
         <origin xyz="0.0096 0.003 0.0" rpy="0 0 0" />
         <mass value="0.015" />
-        <inertia ixx="0.000000200" ixy="0.000000025" ixz="0.000000000"
-                 iyy="0.000000469" iyz="0.000000000" izz="0.000000494" />
+        <inertia ixx="0.001" ixy="0" ixz="0" iyy="0.001" iyz="0" izz="0.001" /> <!-- To stabilize simulation -->
       </inertial>
       <visual>

File: urdf/palm.urdf.xacro (robot description, xacro)
@@ -25,5 +25,6 @@
       <inertial>
         <origin xyz="0.0641 -0.0022 0.0021" rpy="0 0 0" />
-        <mass value="0.598" />
+        <!-- NOTE: Less than total palm mass of 0.598kg because actuator masses are specified separately -->
+        <mass value="0.4" />
         <inertia ixx="0.000305100" ixy="0.000005037" ixz="0.000015302"
                  iyy="0.000811920" iyz="0.000007622" izz="0.000655851" />

Commit message: Fix xacro warnings

File: urdf/actuators.urdf.xacro (robot description, xacro)
@@ -11,5 +11,5 @@
   <xacro:macro name="thumb_actuator" params="name parent *origin">
     <xacro:actuator_impl parent="${parent}" name="${name}">
-      <insert_block name="origin" />
+      <xacro:insert_block name="origin" />
       <limit lower="${-150 * deg_to_rad}" upper="${360 * deg_to_rad}" effort="2.0" velocity="3.35" /> <!-- TODO: Tune effort -->
       <safety_controller k_position="20"
@@ -22,5 +22,5 @@
   <xacro:macro name="index_actuator" params="name parent *origin">
     <xacro:actuator_impl parent="${parent}" name="${name}">
-      <insert_block name="origin" />
+      <xacro:insert_block name="origin" />
       <limit lower="${-175 * deg_to_rad}" upper="${390 * deg_to_rad}" effort="2.0" velocity="3.35" /> <!-- TODO: Tune effort -->
       <safety_controller k_position="20"
@@ -33,5 +33,5 @@
   <xacro:macro name="mrl_actuator" params="name parent *origin">
     <xacro:actuator_impl parent="${parent}" name="${name}">
-      <insert_block name="origin" />
+      <xacro:insert_block name="origin" />
       <limit lower="${-145 * deg_to_rad}" upper="${530 * deg_to_rad}" effort="2.0" velocity="3.56" /> <!-- TODO: Tune effort -->
       <safety_controller k_position="20"
@@ -54,9 +54,9 @@
       <parent link="${parent}" />
       <child link="${name}_link" />
-      <insert_block name="origin" />
+      <xacro:insert_block name="origin" />
       <axis xyz="0 0 1" />
-      <insert_block name="limit" />
+      <xacro:insert_block name="limit" />
       <dynamics friction="0.0" damping="0.5"/> <!-- TODO: Tune -->
-      <insert_block name="safety_controller" />
+      <xacro:insert_block name="safety_controller" />
     </joint>
     <link name="${name}_link">

File: urdf/deg_to_rad.urdf.xacro (robot description, xacro)
@@ -8,4 +8,4 @@
 -->
 <robot xmlns:xacro="http://ros.org/wiki/xacro">
-  <property name="deg_to_rad" value="0.01745329251994329577" />
+  <xacro:property name="deg_to_rad" value="0.01745329251994329577" />
 </robot>

File: urdf/fingers.urdf.xacro (robot description, xacro)
@@ -41,5 +41,5 @@
     <!--Abductor-->
     <xacro:finger_abd parent="${parent}" name="${name}_abd" reflect="${reflect}">
-      <insert_block name="origin" />
+      <xacro:insert_block name="origin" />
     </xacro:finger_abd>
     <!--First flexor-->
@@ -77,5 +77,5 @@
     <!--Abductor-->
     <xacro:thumb_abd parent="${parent}" name="${name}_abd" reflect="${reflect}">
-      <insert_block name="origin" />
+      <xacro:insert_block name="origin" />
     </xacro:thumb_abd>
     <!--First flexor-->
@@ -106,5 +106,5 @@
       <parent link="${parent}" />
       <child link="${name}_link" />
-      <insert_block name="origin" />
+      <xacro:insert_block name="origin" />
       <axis xyz="0 0 1" />
       <limit lower="${finger_abd_min}" upper="${finger_abd_max}" effort="${finger_max_eff}" velocity="${finger_max_vel}" />
@@ -147,5 +147,5 @@
       <parent link="${parent}" />
       <child link="${name}_link" />
-      <insert_block name="origin" />
+      <xacro:insert_block name="origin" />
       <axis xyz="0 0 1" />
       <limit lower="${thumb_abd_min}" upper="${thumb_abd_max}" effort="${finger_max_eff}" velocity="${finger_max_vel}" />
@@ -189,5 +189,5 @@
       <parent link="${parent}" />
       <child link="${name}_link" />
-      <insert_block name="origin" />
+      <xacro:insert_block name="origin" />
       <axis xyz="0 0 1" />
       <limit lower="${finger_flex_min}" upper="${finger_flex_max}" effort="${finger_max_eff}" velocity="${finger_max_vel}" />
@@ -232,5 +232,5 @@
       <parent link="${parent}" />
       <child link="${name}_link" />
-      <insert_block name="origin" />
+      <xacro:insert_block name="origin" />
       <axis xyz="0 0 1" />
       <limit lower="${finger_flex_min}" upper="${finger_flex_max}" effort="${finger_max_eff}" velocity="${finger_max_vel}" />
@@ -275,5 +275,5 @@
       <parent link="${parent}" />
       <child link="${name}_link" />
-      <insert_block name="origin" />
+      <xacro:insert_block name="origin" />
       <axis xyz="0 0 1" />
       <limit lower="${finger_flex_min}" upper="${finger_flex_max}" effort="${finger_max_eff}" velocity="${finger_max_vel}" />

File: urdf/hey5_hand.urdf.xacro (robot description, xacro)
@@ -41,5 +41,5 @@
     </link>
     <joint name="${name}_tool_joint" type="fixed">
-      <insert_block name="origin"/>
+      <xacro:insert_block name="origin"/>
       <parent link="${parent}" />
       <child link="${name}_tool_link" />
@@ -48,5 +48,5 @@
     <!--Palm-->
     <xacro:palm parent="${parent}" name="${name}_palm" reflect="${reflect}" >
-      <insert_block name="origin" />
+      <xacro:insert_block name="origin" />
     </xacro:palm>
     <!--Actuators-->

File: urdf/palm.urdf.xacro (robot description, xacro)
@@ -20,5 +20,5 @@
       <parent link="${parent}" />
       <child link="${name}_link" />
-      <insert_block name="origin" />
+      <xacro:insert_block name="origin" />
     </joint>
     <link name="${name}_link">

Commit message: Remove comments to workaround https://github.com/ros2/launch_ros/issues/214

File: urdf/actuators.urdf.xacro (robot description, xacro)
@@ -12,5 +12,5 @@
     <xacro:actuator_impl parent="${parent}" name="${name}">
       <xacro:insert_block name="origin" />
-      <limit lower="${-150 * deg_to_rad}" upper="${360 * deg_to_rad}" effort="2.0" velocity="3.35" /> <!-- TODO: Tune effort -->
+      <limit lower="${-150 * deg_to_rad}" upper="${360 * deg_to_rad}" effort="2.0" velocity="3.35" />
       <safety_controller k_position="20"
                          k_velocity="20"
@@ -23,5 +23,5 @@
     <xacro:actuator_impl parent="${parent}" name="${name}">
       <xacro:insert_block name="origin" />
-      <limit lower="${-175 * deg_to_rad}" upper="${390 * deg_to_rad}" effort="2.0" velocity="3.35" /> <!-- TODO: Tune effort -->
+      <limit lower="${-175 * deg_to_rad}" upper="${390 * deg_to_rad}" effort="2.0" velocity="3.35" />
       <safety_controller k_position="20"
                          k_velocity="20"
@@ -34,5 +34,5 @@
     <xacro:actuator_impl parent="${parent}" name="${name}">
       <xacro:insert_block name="origin" />
-      <limit lower="${-145 * deg_to_rad}" upper="${530 * deg_to_rad}" effort="2.0" velocity="3.56" /> <!-- TODO: Tune effort -->
+      <limit lower="${-145 * deg_to_rad}" upper="${530 * deg_to_rad}" effort="2.0" velocity="3.56" />
       <safety_controller k_position="20"
                          k_velocity="20"
@@ -57,5 +57,5 @@
       <axis xyz="0 0 1" />
       <xacro:insert_block name="limit" />
-      <dynamics friction="0.0" damping="0.5"/> <!-- TODO: Tune -->
+      <dynamics friction="0.0" damping="0.5"/>
       <xacro:insert_block name="safety_controller" />
     </joint>

File: urdf/fingers.urdf.xacro (robot description, xacro)
@@ -14,12 +14,12 @@
   <xacro:property name="thumb_abd_min"   value="${  0 * deg_to_rad}" />
   <xacro:property name="thumb_abd_max"   value="${ 90 * deg_to_rad}" />
-  <xacro:property name="finger_abd_min"  value="${-30 * deg_to_rad}" /> <!--TODO: Check-->
-  <xacro:property name="finger_abd_max"  value="${ 30 * deg_to_rad}" /> <!--TODO: Check-->
+  <xacro:property name="finger_abd_min"  value="${-30 * deg_to_rad}" />
+  <xacro:property name="finger_abd_max"  value="${ 30 * deg_to_rad}" />
   <xacro:property name="finger_flex_min" value="${  0 * deg_to_rad}" />
   <xacro:property name="finger_flex_max" value="${ 45 * deg_to_rad}" />
-  <xacro:property name="finger_max_vel"  value="2.0" />                 <!--TODO: Check-->
-  <xacro:property name="finger_max_eff"  value="2.0" />                 <!--TODO: Check-->
-  <xacro:property name="finger_friction" value="0.0" />                 <!--TODO: Check-->
-  <xacro:property name="finger_damping"  value="0.5" />                 <!--TODO: Check-->
+  <xacro:property name="finger_max_vel"  value="2.0" />
+  <xacro:property name="finger_max_eff"  value="2.0" />
+  <xacro:property name="finger_friction" value="0.0" />
+  <xacro:property name="finger_damping"  value="0.5" />
   <xacro:property name="finger_d1"  value="0.009" />
   <xacro:property name="finger_d2"  value="0.013" />
@@ -197,5 +197,5 @@
       <inertial>
         <origin xyz="${finger_d2 / 2.0} 0 0" rpy="0 0 0" />
-        <mass value="0.01" /> <!--TODO: can we make it zero and still have a stable dynamic simulation?-->
+        <mass value="0.01" />
         <inertia ixx="0.001" ixy="0" ixz="0" iyy="0.001" iyz="0" izz="0.001" /> <!-- To stabilize simulation -->
       </inertial>

File: urdf/palm.urdf.xacro (robot description, xacro)
@@ -25,5 +25,4 @@
       <inertial>
         <origin xyz="0.0641 -0.0022 0.0021" rpy="0 0 0" />
-        <!-- NOTE: Less than total palm mass of 0.598kg because actuator masses are specified separately -->
         <mass value="0.4" />
         <inertia ixx="0.000305100" ixy="0.000005037" ixz="0.000015302"
