Commit message: Fix hay5 hand for REEM-C robot

File: gazebo/gazebo.urdf.xacro (robot description, xacro)
@@ -8,4 +8,8 @@
 -->
 <robot xmlns:xacro="http://ros.org/wiki/xacro">
+   <xacro:arg name="multiple" default="false"/>
+   <xacro:arg name="namespace" default=""/>
+   <xacro:property name="is_multiple" value="$(arg multiple)" />
+   <xacro:property name="nsp" value="$(arg namespace)" />
    <xacro:macro name="hey5_gazebo_simulation" params="side">
    <gazebo>
